File: Circuit/boneIO - input board/boneIO_input board.sch (KiCad schematic (older format))
At the start: 262 parts, among them J1 Screw_Terminal_01x08, J10 Screw_Terminal_01x08, J11 Screw_Terminal_01x08, J12 ZW_VCC, J13 ZW_GND, J14 INNY ZASILACZ, J15 BeagleBone_Black_Header, J16 BeagleBone_Black_Header, J2 Screw_Terminal_01x08, J3 Screw_Terminal_01x08, J4 Screw_Terminal_01x08, J5 Screw_Terminal_01x08, J6 Screw_Terminal_01x08, J7 Screw_Terminal_01x08, J8 Screw_Terminal_01x04, J9 Conn_02x04_Odd_Even, SW1 SW_Push, U1 P82B96, U10 LM2596S-ADJ, U11 RS485, U12 PC817X2NIP0F, U13 PC817X2NIP0F, U14 PC817X2NIP0F, U15 PC817X2NIP0F, U16 PC817X2NIP0F, U17 PC817X2NIP0F, U18 PC817X2NIP0F, U19 PC817X2NIP0F, U2 PC817X2NIP0F, U20 PC817X2NIP0F, U21 PC817X2NIP0F, U22 PC817X2NIP0F, U23 PC817X2NIP0F, U24 PC817X2NIP0F, U25 PC817X2NIP0F, U26 PC817X2NIP0F, U27 PC817X2NIP0F, U28 PC817X2NIP0F, U29 PC817X2NIP0F, U3 PC817X2NIP0F, U30 PC817X2NIP0F, U31 PC817X2NIP0F, U32 PC817X2NIP0F, U33 PC817X2NIP0F, U34 PC817X2NIP0F, U35 PC817X2NIP0F, U36 DS1307Z+, U37 PC817X2NIP0F, U38 PC817X2NIP0F, U39 PC817X2NIP0F, U4 PC817X2NIP0F, U40 PC817X2NIP0F, U41 PC817X2NIP0F, U42 PC817X2NIP0F, U43 PC817X2NIP0F, U44 PC817X2NIP0F, U45 PC817X2NIP0F, U46 PC817X2NIP0F, U47 PC817X2NIP0F, U48 PC817X2NIP0F, U49 PC817X2NIP0F, U5 PC817X2NIP0F, U50 PC817X2NIP0F, U51 PC817X2NIP0F, U52 PC817X2NIP0F, U53 PC817X2NIP0F, U54 PC817X2NIP0F, U55 PC817X2NIP0F, U56 PC817X2NIP0F, U6 PC817X2NIP0F, U7 PC817X2NIP0F, U8 PC817X2NIP0F, U9 PC817X2NIP0F, Y1 32,788 MHz

Commit message: Correction of a schematic error and repair of 3d models
Connections:
- net GNDA: now also U12.2, U13.2, U14.2, U15.2, U16.2, U17.2, U18.2, U19.2, U2.2, U20.2, U21.2, U22.2, U23.2, U24.2, U25.2, U26.2, U27.2, U28.2, U29.2, U3.2, U30.2, U31.2, U32.2, U33.2, U34.2, U35.2, U37.2, U38.2, U39.2, U4.2, U40.2, U41.2, U42.2, U43.2, U44.2, U45.2, U46.2, U47.2, U48.2, U49.2, U5.2, U50.2, U51.2, U52.2, U53.2, U54.2, U55.2, U56.2, U6.2, U7.2, U8.2, U9.2; no longer R1.2, R100.2, R109.2, R110.2, R111.2, R112.2, R2.2, R21.2, R22.2, R23.2, R24.2, R25.2, R26.2, R27.2, R28.2, R3.2, R4.2, R40.2, R41.2, R42.2, R43.2, R44.2, R45.2, R46.2, R47.2, R5.2, R58.2, R59.2, R6.2, R60.2, R61.2, R62.2, R63.2, R64.2, R65.2, R7.2, R77.2, R78.2, R79.2, R8.2, R80.2, R81.2, R82.2, R83.2, R84.2, R93.2, R94.2, R95.2, R96.2, R97.2, R98.2, R99.2
- net P8.07_OUT: now also R109.2; no longer U53.2
- net P8.08_OUT: now also R61.2; no longer U31.2
- net P8.09_OUT: now also R62.2; no longer U32.2
- net P8.10_OUT: now also R63.2; no longer U33.2
- net P8.11_OUT: now also R64.2; no longer U34.2
- net P8.12_OUT: now also R65.2; no longer U35.2
- net P8.13_OUT: now also R97.2; no longer U49.2
- net P8.14_OUT: now also R46.2; no longer U26.2
- net P8.15_OUT: now also R47.2; no longer U27.2
- net P8.16_OUT: now also R58.2; no longer U28.2
- net P8.17_OUT: now also R60.2; no longer U30.2
- net P8.18_OUT: now also R59.2; no longer U29.2
- net P8.19_OUT: now also R79.2; no longer U39.2
- net P8.26_OUT: now also R43.2; no longer U23.2
- net P8.27_OUT: now also R42.2; no longer U22.2
- net P8.28_OUT: now also R41.2; no longer U21.2
- net P8.29_OUT: now also R40.2; no longer U20.2
- net P8.30_OUT: now also R28.2; no longer U19.2
- net P8.31_OUT: now also R27.2; no longer U18.2
- net P8.32_OUT: now also R26.2; no longer U17.2
- net P8.33_OUT: now also R25.2; no longer U16.2
- net P8.34_OUT: now also R24.2; no longer U15.2
- net P8.35_OUT: now also R23.2; no longer U14.2
- net P8.36_OUT: now also R22.2; no longer U13.2
- net P8.37_OUT: now also R21.2; no longer U12.2
- net P8.38_OUT: now also R8.2; no longer U9.2
- net P8.39_OUT: now also R7.2; no longer U8.2
- net P8.40_OUT: now also R6.2; no longer U7.2
- net P8.41_OUT: now also R5.2; no longer U6.2
- net P8.42_OUT: now also R4.2; no longer U5.2
- net P8.43_OUT: now also R3.2; no longer U4.2
- net P8.44_OUT: now also R2.2; no longer U3.2
- net P8.45_OUT: now also R1.2; no longer U2.2
- net P8.46_OUT: now also R100.2; no longer U52.2
- net P9.11_OUT: now also R81.2; no longer U41.2
- net P9.12_OUT: now also R82.2; no longer U42.2
- net P9.13_OUT: now also R83.2; no longer U43.2
- net P9.14_OUT: now also R84.2; no longer U44.2
- net P9.15_OUT: now also R44.2; no longer U24.2
- net P9.16_OUT: now also R45.2; no longer U25.2
- net P9.17_OUT: now also R99.2; no longer U51.2
- net P9.18_OUT: now also R94.2; no longer U46.2
- net P9.21_OUT: now also R95.2; no longer U47.2
- net P9.22_OUT: now also R96.2; no longer U48.2
- net P9.23_OUT: now also R98.2; no longer U50.2
- net P9.25_OUT: now also R80.2; no longer U40.2
- net P9.27_OUT: now also R78.2; no longer U38.2
- net P9.28_OUT: now also R77.2; no longer U37.2
- net P9.29_OUT: now also R93.2; no longer U45.2
- net P9.30_OUT: now also R112.2; no longer U56.2
- net P9.31_OUT: now also R111.2; no longer U55.2
- net P9.42_OUT: now also R110.2; no longer U54.2
