File: Circuit/boneIO - input board/boneIO_input board.sch (KiCad schematic (older format))
At the start: 262 parts, among them J1 Screw_Terminal_01x08, J10 Screw_Terminal_01x08, J11 Screw_Terminal_01x08, J12 ZW_VCC, J13 ZW_GND, J14 INNY ZASILACZ, J15 BeagleBone_Black_Header, J16 BeagleBone_Black_Header, J2 Screw_Terminal_01x08, J3 Screw_Terminal_01x08, J4 Screw_Terminal_01x08, J5 Screw_Terminal_01x08, J6 Screw_Terminal_01x08, J7 Screw_Terminal_01x08, J8 Screw_Terminal_01x04, J9 Conn_02x04_Odd_Even, SW1 SW_Push, U1 P82B96, U10 LM2596S-ADJ, U11 RS485, U12 PC817X2NIP0F, U13 PC817X2NIP0F, U14 PC817X2NIP0F, U15 PC817X2NIP0F, U16 PC817X2NIP0F, U17 PC817X2NIP0F, U18 PC817X2NIP0F, U19 PC817X2NIP0F, U2 PC817X2NIP0F, U20 PC817X2NIP0F, U21 PC817X2NIP0F, U22 PC817X2NIP0F, U23 PC817X2NIP0F, U24 PC817X2NIP0F, U25 PC817X2NIP0F, U26 PC817X2NIP0F, U27 PC817X2NIP0F, U28 PC817X2NIP0F, U29 PC817X2NIP0F, U3 PC817X2NIP0F, U30 PC817X2NIP0F, U31 PC817X2NIP0F, U32 PC817X2NIP0F, U33 PC817X2NIP0F, U34 PC817X2NIP0F, U35 PC817X2NIP0F, U36 DS1307Z+, U37 PC817X2NIP0F, U38 PC817X2NIP0F, U39 PC817X2NIP0F, U4 PC817X2NIP0F, U40 PC817X2NIP0F, U41 PC817X2NIP0F, U42 PC817X2NIP0F, U43 PC817X2NIP0F, U44 PC817X2NIP0F, U45 PC817X2NIP0F, U46 PC817X2NIP0F, U47 PC817X2NIP0F, U48 PC817X2NIP0F, U49 PC817X2NIP0F, U5 PC817X2NIP0F, U50 PC817X2NIP0F, U51 PC817X2NIP0F, U52 PC817X2NIP0F, U53 PC817X2NIP0F, U54 PC817X2NIP0F, U55 PC817X2NIP0F, U56 PC817X2NIP0F, U6 PC817X2NIP0F, U7 PC817X2NIP0F, U8 PC817X2NIP0F, U9 PC817X2NIP0F, Y1 32,788 MHz

Commit message: relay board v0.3 and some cleanup
Parts:
- removed J12: ZW_VCC, Connector_PinHeader_2.54mm:PinHeader_1x03_P2.54mm_Vertical, symbol Connector:Screw_Terminal_01x03
- removed J13: ZW_GND, Connector_PinHeader_2.54mm:PinHeader_1x03_P2.54mm_Vertical, symbol Connector:Screw_Terminal_01x03
- removed J14: INNY ZASILACZ, Connector:Phoenix_1x02_P5.00mm_Horizontal, symbol Connector:Screw_Terminal_01x02
- removed R108, R11: 10k, Resistor_SMD:R_0603_1608Metric, symbol Device:R
- added C38: 100n, Capacitor_SMD:C_0603_1608Metric, symbol Device:C
- added J4: ZASILACZ, Connector_Phoenix_MSTB:PhoenixContact_MSTBA_2,5_2-G_1x02_P5.00mm_Horizontal, symbol Connector:Screw_Terminal_01x02
- added L3, L4: BLM21PG221SN1D, Inductor_SMD:L_0805_2012Metric, symbol Device:L
- added Q1, Q2: BSS138, Package_TO_SOT_SMD:SOT-23, symbol Transistor_FET:BSS138
- added R103, R104, R109, R110, R111, R112: 10k, Resistor_SMD:R_0603_1608Metric, symbol Device:R
- added R121, R122, R123, R124, R125, R126: 4.7k, Resistor_SMD:R_0603_1608Metric, symbol Device:R
- added U51, U52, U57, U58, U59, U60: PC817X2NIP0F, PC817:SOT254P975X400-4N, symbol Isolator:PC817
- BT1: footprint boneIO:Battery_Panasonic_CR1220-VCN_Vertical_CircularHoles -> Battery:Battery_Panasonic_CR1220-VCN_Vertical_CircularHoles
- I2C1: value Conn_01x04 -> OLED
- J11: renamed from J15; symbol boneIO:BeagleBone_Black_Header-Connector_Generic-boneIO_input-board_v0.3-rescue-boneIO_input-board-rescue -> Connector_Generic:Conn_02x23_Odd_Even
- J12: renamed from J16; symbol boneIO:BeagleBone_Black_Header-Connector_Generic-boneIO_input-board_v0.3-rescue-boneIO_input-board-rescue -> Connector_Generic:Conn_02x23_Odd_Even
- R68: renamed from R66; value 10k -> 4.7k
- R69: renamed from R67; value 10k -> 4.7k
- U1: renamed from U52; footprint boneIO - RM85:SOT254P975X400-4N -> PC817:SOT254P975X400-4N
- U10: renamed from U9; footprint boneIO - RM85:SOT254P975X400-4N -> PC817:SOT254P975X400-4N
- U11: renamed from U12; footprint boneIO - RM85:SOT254P975X400-4N -> PC817:SOT254P975X400-4N
- U12: renamed from U13; footprint boneIO - RM85:SOT254P975X400-4N -> PC817:SOT254P975X400-4N
- U13: renamed from U14; footprint boneIO - RM85:SOT254P975X400-4N -> PC817:SOT254P975X400-4N
- U14: renamed from U15; footprint boneIO - RM85:SOT254P975X400-4N -> PC817:SOT254P975X400-4N
- U15: renamed from U16; footprint boneIO - RM85:SOT254P975X400-4N -> PC817:SOT254P975X400-4N
- U16: renamed from U17; footprint boneIO - RM85:SOT254P975X400-4N -> PC817:SOT254P975X400-4N
- U17: renamed from U18; footprint boneIO - RM85:SOT254P975X400-4N -> PC817:SOT254P975X400-4N
- U18: renamed from U39; footprint boneIO - RM85:SOT254P975X400-4N -> PC817:SOT254P975X400-4N
- U19: renamed from U29; footprint boneIO - RM85:SOT254P975X400-4N -> PC817:SOT254P975X400-4N
- U2, U27, U3, U4, U5, U55, U6, U7, U8: footprint boneIO - RM85:SOT254P975X400-4N -> PC817:SOT254P975X400-4N
- U20: renamed from U30; footprint boneIO - RM85:SOT254P975X400-4N -> PC817:SOT254P975X400-4N
- U21: renamed from U19; footprint boneIO - RM85:SOT254P975X400-4N -> PC817:SOT254P975X400-4N
- U22: renamed from U20; footprint boneIO - RM85:SOT254P975X400-4N -> PC817:SOT254P975X400-4N
- U23: renamed from U21; footprint boneIO - RM85:SOT254P975X400-4N -> PC817:SOT254P975X400-4N
- U24: renamed from U22; footprint boneIO - RM85:SOT254P975X400-4N -> PC817:SOT254P975X400-4N
- U25: renamed from U23; footprint boneIO - RM85:SOT254P975X400-4N -> PC817:SOT254P975X400-4N
- U26: renamed from U28; footprint boneIO - RM85:SOT254P975X400-4N -> PC817:SOT254P975X400-4N
- U28: renamed from U26; footprint boneIO - RM85:SOT254P975X400-4N -> PC817:SOT254P975X400-4N
- U29: renamed from U49; footprint boneIO - RM85:SOT254P975X400-4N -> PC817:SOT254P975X400-4N
- U30: renamed from U35; footprint boneIO - RM85:SOT254P975X400-4N -> PC817:SOT254P975X400-4N
- U31: renamed from U34; footprint boneIO - RM85:SOT254P975X400-4N -> PC817:SOT254P975X400-4N
- U32: renamed from U33; footprint boneIO - RM85:SOT254P975X400-4N -> PC817:SOT254P975X400-4N
- U33: renamed from U32; footprint boneIO - RM85:SOT254P975X400-4N -> PC817:SOT254P975X400-4N
- U35: renamed from U31; footprint boneIO - RM85:SOT254P975X400-4N -> PC817:SOT254P975X400-4N
- U36: renamed from U53; footprint boneIO - RM85:SOT254P975X400-4N -> PC817:SOT254P975X400-4N
- U37: renamed from U41; footprint boneIO - RM85:SOT254P975X400-4N -> PC817:SOT254P975X400-4N
- U38: renamed from U42; footprint boneIO - RM85:SOT254P975X400-4N -> PC817:SOT254P975X400-4N
- U39: renamed from U43; footprint boneIO - RM85:SOT254P975X400-4N -> PC817:SOT254P975X400-4N
- U40: renamed from U44; footprint boneIO - RM85:SOT254P975X400-4N -> PC817:SOT254P975X400-4N
- U41: renamed from U24; footprint boneIO - RM85:SOT254P975X400-4N -> PC817:SOT254P975X400-4N
- U42: renamed from U25; footprint boneIO - RM85:SOT254P975X400-4N -> PC817:SOT254P975X400-4N
- U43: renamed from U51; footprint boneIO - RM85:SOT254P975X400-4N -> PC817:SOT254P975X400-4N
- U44: renamed from U46; footprint boneIO - RM85:SOT254P975X400-4N -> PC817:SOT254P975X400-4N
- U45: renamed from U47; footprint boneIO - RM85:SOT254P975X400-4N -> PC817:SOT254P975X400-4N
- U46: renamed from U48; footprint boneIO - RM85:SOT254P975X400-4N -> PC817:SOT254P975X400-4N
- U47: renamed from U50; footprint boneIO - RM85:SOT254P975X400-4N -> PC817:SOT254P975X400-4N
- U48: renamed from U40; footprint boneIO - RM85:SOT254P975X400-4N -> PC817:SOT254P975X400-4N
- U49: renamed from U38; footprint boneIO - RM85:SOT254P975X400-4N -> PC817:SOT254P975X400-4N
- U50: renamed from U37; footprint boneIO - RM85:SOT254P975X400-4N -> PC817:SOT254P975X400-4N
- U53: renamed from U45; footprint boneIO - RM85:SOT254P975X400-4N -> PC817:SOT254P975X400-4N
- U54: renamed from U56; footprint boneIO - RM85:SOT254P975X400-4N -> PC817:SOT254P975X400-4N
- U56: renamed from U54; footprint boneIO - RM85:SOT254P975X400-4N -> PC817:SOT254P975X400-4N
- U61: renamed from U11; footprint Module:RS485_moduleTTL -> rs485:RS485_moduleTTL; symbol boneIO:RS485-RF_Module-boneIO_input-board_v0.3-rescue-boneIO_input-board-rescue -> RS485:RS485_module
- renumbered C2 to C1, C12 to C11, C13 to C12, C11 to C13, C3 to C2, C41 to C21, C32 to C22, C33 to C23, C21 to C24, C23 to C25, C24 to C26, C25 to C27, C26 to C28, C22 to C29, C54 to C3, C31 to C30, C30 to C31, C29 to C32, C51 to C33, C38 to C34, C37 to C35, C35 to C37, C34 to C39, C55 to C40, C43 to C41, C44 to C42, C45 to C43, C46 to C44, C27 to C45, C28 to C46, C53 to C47, C52 to C51, C42 to C52, C40 to C53, C39 to C54, C47 to C55, C58 to C56, C56 to C58, C1 to C59, D3 to D2, D4 to D3, D5 to D4, D2 to D5, J11 to J1, J8 to J10, J9 to J13, J10 to J14, J1 to J2, J2 to J3, J3 to J5, J4 to J6, J5 to J7, J6 to J8, J7 to J9, R100 to R1, R13 to R10, R88 to R100, R86 to R101, R85 to R102, R93 to R105, R112 to R106, R111 to R107, R110 to R108, R14 to R11, R101 to R113, R116 to R114, R114 to R116, R56 to R117, R57 to R118, R9 to R119, R15 to R12, R10 to R120, R16 to R13, R17 to R14, R8 to R15, R21 to R16, R22 to R17, R23 to R18, R24 to R19, R1 to R2, R25 to R20, R26 to R21, R27 to R22, R19 to R23, R20 to R24, R29 to R25, R18 to R26, R30 to R27, R31 to R28, R32 to R29, R2 to R3, R33 to R30, R34 to R31, R35 to R32, R36 to R33, R79 to R34, R59 to R35, R60 to R36, R28 to R37, R40 to R38, R41 to R39, R3 to R4, R42 to R40, R43 to R41, R38 to R42, R87 to R43, R69 to R44, R70 to R45, R37 to R46, R48 to R47, R49 to R48, R50 to R49, R4 to R5, R51 to R50, R39 to R51, R58 to R52, R47 to R53, R46 to R54, R97 to R55, R65 to R56, R64 to R57, R63 to R58, R62 to R59, R5 to R6, R68 to R60, R55 to R61, R54 to R62, R105 to R63, R75 to R64, R74 to R65, R73 to R66, R72 to R67, R6 to R7, R61 to R70, R109 to R71, R81 to R72, R82 to R73, R83 to R74, R84 to R75, R44 to R76, R45 to R77, R76 to R78, R71 to R79, R7 to R8, R113 to R80, R89 to R81, R90 to R82, R91 to R83, R92 to R84, R52 to R85, R53 to R86, R99 to R87, R94 to R88, R95 to R89, R12 to R9, R96 to R90, R98 to R91, R80 to R92, R78 to R93, R77 to R94, R107 to R95, R102 to R96, R103 to R97, R104 to R98, R106 to R99, U36 to U34, U1 to U62, U10 to U9
Connections:
- net +24V: now also R109.1, R111.1, U51.3
- net +3V3: now also R121.1, R122.1, R123.1, R124.1; no longer R68.1, R69.1, R78.1, U34.8 (VCC)
- net +48V: now also J4.2 (Pin_2), R103.1, R104.1, R110.1, R112.1, U57.3
- net +5V: now also R68.1, R69.1, R78.1, U34.8 (VCC), C38.1, R125.1, R126.1
- net GND: now also C38.2, U51.2, U52.3, U58.3, U60.2, U60.3
- net GND1: now also J4.1 (Pin_1), U52.2, U57.2, U58.2, U59.2, U59.3
- net GNDA: now also L4.2
- net SCL: now also Q2.2 (S), R122.2; no longer R69.2, U34.6 (SCL)
- net SDA: now also Q1.2 (S), R121.2; no longer R68.2, U34.5 (SDA)
- net VDD: now also L3.2
- net GNDD renamed GND2
- net P8.03: no longer names the net of J12.3 (Pin_3)
- net P8.04: no longer names the net of J12.4 (Pin_4)
- net P8.05: no longer names the net of J12.5 (Pin_5)
- net P8.06: no longer names the net of J12.6 (Pin_6)
- net P8.20: no longer names the net of J12.20 (Pin_20)
- net P8.21: no longer names the net of J12.21 (Pin_21)
- net P8.22: no longer names the net of J12.22 (Pin_22)
- net P8.23: no longer names the net of J12.23 (Pin_23)
- net P8.24: no longer names the net of J12.24 (Pin_24)
- net P8.25: no longer names the net of J12.25 (Pin_25)
- new net: L4.1, U59.4, U60.4
- new net: R103.2, U52.1
- new net: R109.2, U51.1, U52.4
- new net: R104.2, U58.1
- new net: R111.2, U58.4, U60.1
- new net: L3.1, U51.4, U57.4
- new net: R110.2, U57.1
- new net: Q1.1 (G), R123.2
- new net: R112.2, U59.1
- new net: Q2.1 (G), R124.2
- new net SCL_5V: Q2.3 (D), R126.2, R69.2, U34.6 (SCL)
- new net SDA_5V: Q1.3 (D), R125.2, R68.2, U34.5 (SDA)
- no-connect marks 1 -> 15
Other:
- note added: "Automatic Power Change\n\n\n"
- note added: "Input Board v0.3 BBB\n\n\n"
- note added: "Logic Level Converter"
- note added: "PINOUT_ RS485_ I2C\n\n\n\n\n"
- note removed: "Input Board v0.2 BBB\n\n\n"
- note removed: "Jumper\n\n\n\n"
- moved on the sheet: BT1, C29, C59, D4, D5, I2C1, J10, J13, J14, J2, J3, J5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
