File: Circuit/boneIO - input board_ESP/boneIO - input board ESP.kicad_pcb (KiCad board)
At the start: 2 copper layers, 207 x 74 mm, 334 parts, among them J1 UART, J10 P2, J11 P4, J12 P6, J13 ZASILACZ, J2 POWER, J3 HR911105A, J4 USB_B_Mini, J5 Conn_02x04_Odd_Even, J6 P1, J7 P3, J8 P5, J9 P7, Q1 AO3401A, Q10 BC817, Q11 BC807, Q12 BC817, Q13 BC807, Q2 BC847, Q3 BSS138, Q4 AO3401A, Q5 BC817, Q6 BC817, Q9 BC817, SW1 SW_Push, SW2 SUPLA_SWITCH, U1 MP1584EN_module, U10 MAX485E, U11 INA226, U12 PC817X2NIP0F, U13 PC817X2NIP0F, U14 PC817X2NIP0F, U15 PC817X2NIP0F, U16 PC817X2NIP0F, U17 PC817X2NIP0F, U18 PC817X2NIP0F, U19 PC817X2NIP0F, U2 AMS1117-3.3, U20 PC817X2NIP0F, U21 PC817X2NIP0F, U22 PC817X2NIP0F, U23 PC817X2NIP0F, U24 PC817X2NIP0F, U25 PC817X2NIP0F, U26 PC817X2NIP0F, U27 PC817X2NIP0F, U28 PC817X2NIP0F, U29 PC817X2NIP0F, U3 LAN8720A, U30 PC817X2NIP0F, U31 PC817X2NIP0F, U32 PC817X2NIP0F, U33 PC817X2NIP0F, U34 PC817X2NIP0F, U35 PC817X2NIP0F, U36 PC817X2NIP0F, U37 PC817X2NIP0F, U38 PC817X2NIP0F, U39 PC817X2NIP0F, U4 MP1584EN, U40 PC817X2NIP0F, U41 PC817X2NIP0F, U42 MCP23017_SS, U43 MCP23017_SS, U44 PC817X2NIP0F, U45 PC817X2NIP0F, U46 PC817X2NIP0F, U47 PC817X2NIP0F, U48 PC817X2NIP0F, U49 PC817X2NIP0F, U5 CH340G, U50 PC817X2NIP0F, U51 PC817X2NIP0F, U52 PC817X2NIP0F, U53 PC817X2NIP0F, U54 PC817X2NIP0F, U6 ESP32-WROOM-32D, U7 P82B96, U8 CD4053B, U9 ISO7220A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

Commit message: update
Parts:
- removed R147, R148, R149, R150, R151, R152: 4.7k, Resistor_SMD:R_0603_1608Metric
- added A0: NO, Jumper:SolderJumper-2_P1.3mm_Open_RoundedPad1.0x1.5mm, F.Cu at (191.2, -28.0)
- added A0: NO, Jumper:SolderJumper-2_P1.3mm_Open_RoundedPad1.0x1.5mm, F.Cu at (142.2, -22.2)
- added A1: NO, Jumper:SolderJumper-2_P1.3mm_Open_RoundedPad1.0x1.5mm, F.Cu at (188.9, -28.0)
- added A1: NO, Jumper:SolderJumper-2_P1.3mm_Open_RoundedPad1.0x1.5mm, F.Cu at (142.2, -19.9)
- added A2: NO, Jumper:SolderJumper-2_P1.3mm_Open_RoundedPad1.0x1.5mm, F.Cu at (186.6, -28.0)
- added A2: NO, Jumper:SolderJumper-2_P1.3mm_Open_RoundedPad1.0x1.5mm, F.Cu at (142.2, -17.8)
- added G***: LOGO, Symbol:boneIO_LOGO_srednie, F.Cu at (107.5, -20.4)
- R153, R154, R155, R156, R157, R158: value 4.7k -> 10k
Connections:
- net GPIO39_ONLY_INPUT renamed Net-(U6-Pad5)
Routing:
- net Net-(JP7-Pad2): track 20.1 -> 24.5 mm
- net Net-(JP5-Pad2): track 22.9 -> 27.3 mm
- net Net-(JP6-Pad2): track 21.0 -> 24.6 mm
- net +3V3: track 605.8 -> 603.6 mm, vias 55 -> 54
- net Net-(JP4-Pad2): track 11.3 -> 12.8 mm
- net Net-(R134-Pad2): track 14.6 -> 14.0 mm
- net Net-(JP2-Pad2): track 12.6 -> 13.2 mm, vias 0 -> 2
- net Net-(JP3-Pad2): track 11.1 -> 11.5 mm, vias 0 -> 2
- net GND: vias 176 -> 180
- added copper zone on F.Cu, net Net-(C20-Pad1)
- added copper zone on F.Cu, net Net-(C9-Pad1)
- removed copper zone on B.Cu, net (none)
Other:
- outline, holes or cut-outs redrawn
