File: Circuit/boneIO - input board_ESP/boneIO - input board ESP.sch (KiCad schematic (older format))
At the start: 334 parts, among them J1 UART, J10 P2, J11 P4, J12 P6, J13 ZASILACZ, J2 POWER, J3 HR911105A, J4 USB_B_Mini, J5 Conn_02x04_Odd_Even, J6 P1, J7 P3, J8 P5, J9 P7, Q1 AO3401A, Q10 BC817, Q11 BC807, Q12 BC817, Q13 BC807, Q2 BC847, Q3 BSS138, Q4 AO3401A, Q5 BC817, Q6 BC817, Q9 BC817, SW1 SW_Push, SW2 SUPLA_SWITCH, U1 MP1584EN_module, U10 MAX485E, U11 INA226, U12 PC817X2NIP0F, U13 PC817X2NIP0F, U14 PC817X2NIP0F, U15 PC817X2NIP0F, U16 PC817X2NIP0F, U17 PC817X2NIP0F, U18 PC817X2NIP0F, U19 PC817X2NIP0F, U2 AMS1117-3.3, U20 PC817X2NIP0F, U21 PC817X2NIP0F, U22 PC817X2NIP0F, U23 PC817X2NIP0F, U24 PC817X2NIP0F, U25 PC817X2NIP0F, U26 PC817X2NIP0F, U27 PC817X2NIP0F, U28 PC817X2NIP0F, U29 PC817X2NIP0F, U3 LAN8720A, U30 PC817X2NIP0F, U31 PC817X2NIP0F, U32 PC817X2NIP0F, U33 PC817X2NIP0F, U34 PC817X2NIP0F, U35 PC817X2NIP0F, U36 PC817X2NIP0F, U37 PC817X2NIP0F, U38 PC817X2NIP0F, U39 PC817X2NIP0F, U4 MP1584EN, U40 PC817X2NIP0F, U41 PC817X2NIP0F, U42 MCP23017_SS, U43 MCP23017_SS, U44 PC817X2NIP0F, U45 PC817X2NIP0F, U46 PC817X2NIP0F, U47 PC817X2NIP0F, U48 PC817X2NIP0F, U49 PC817X2NIP0F, U5 CH340G, U50 PC817X2NIP0F, U51 PC817X2NIP0F, U52 PC817X2NIP0F, U53 PC817X2NIP0F, U54 PC817X2NIP0F, U6 ESP32-WROOM-32D, U7 P82B96, U8 CD4053B, U9 ISO7220A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

Commit message: update
Parts:
- removed R147, R148, R149, R150, R151, R152: 4.7k, Resistor_SMD:R_0603_1608Metric, symbol Device:R
- added JP2, JP3, JP4, JP5, JP6, JP7: NO, Jumper:SolderJumper-2_P1.3mm_Open_RoundedPad1.0x1.5mm, symbol Device:Jumper_NO_Small
- R153, R154, R155, R156, R157, R158: value 4.7k -> 10k
Connections:
- net +3V3: now also JP2.1, JP3.1, JP4.1, JP5.1, JP6.1, JP7.1
- net at R155.1, U42.15 (A0): now also JP4.2
- net at R154.1, U42.16 (A1): now also JP3.2
- net at R153.1, U42.17 (A2): now also JP2.2
- net at R158.1, U43.15 (A0): now also JP7.2
- net at R157.1, U43.16 (A1): now also JP6.2
- net at R156.1, U43.17 (A2): now also JP5.2
Changed lines of the file:
@@
 	29350 20000 29100 20000
 $Comp
-L Device:R R152
-U 1 1 6973B9C8
-P 28800 19900
-F 0 "R152" H 28870 19946 50  0000 L CNN
-F 1 "4.7k" H 28870 19855 50  0000 L CNN
-F 2 "Resistor_SMD:R_0603_1608Metric" V 28730 19900 50  0001 C CNN
-F 3 "~" H 28800 19900 50  0001 C CNN
-	1    28800 19900
-	1    0    0    -1
-$EndComp
-$Comp
-L Device:R R151
-U 1 1 69A46D35
-P 28500 19900
-F 0 "R151" H 28570 19946 50  0000 L CNN
-F 1 "4.7k" H 28570 19855 50  0000 L CNN
-F 2 "Resistor_SMD:R_0603_1608Metric" V 28430 19900 50  0001 C CNN
-F 3 "~" H 28500 19900 50  0001 C CNN
-	1    28500 19900
-	1    0    0    -1
-$EndComp
-$Comp
-L Device:R R150
-U 1 1 69BCC633
-P 28200 19900
-F 0 "R150" H 28270 19946 50  0000 L CNN
-F 1 "4.7k" H 28270 19855 50  0000 L CNN
-F 2 "Resistor_SMD:R_0603_1608Metric" V 28130 19900 50  0001 C CNN
-F 3 "~" H 28200 19900 50  0001 C CNN
-	1    28200 19900
-	1    0    0    -1
-$EndComp
-$Comp
 L Device:R R156
 U 1 1 69D51E23
 P 28200 20450
 F 0 "R156" H 28270 20496 50  0000 L CNN
-F 1 "4.7k" H 28270 20405 50  0000 L CNN
+F 1 "10k" H 28270 20405 50  0000 L CNN
 F 2 "Resistor_SMD:R_0603_1608Metric" V 28130 20450 50  0001 C CNN
 F 3 "~" H 28200 20450 50  0001 C CNN
@@
 P 28500 20450
 F 0 "R157" H 28570 20496 50  0000 L CNN
-F 1 "4.7k" H 28570 20405 50  0000 L CNN
+F 1 "10k" H 28570 20405 50  0000 L CNN
 F 2 "Resistor_SMD:R_0603_1608Metric" V 28430 20450 50  0001 C CNN
 F 3 "~" H 28500 20450 50  0001 C CNN
@@
 P 28800 20450
 F 0 "R158" H 28870 20496 50  0000 L CNN
-F 1 "4.7k" H 28870 20405 50  0000 L CNN
+F 1 "10k" H 28870 20405 50  0000 L CNN
 F 2 "Resistor_SMD:R_0603_1608Metric" V 28730 20450 50  0001 C CNN
 F 3 "~" H 28800 20450 50  0001 C CNN
@@
 	29100 20100 28200 20100
 Wire Wire Line
-	28200 20100 28200 20050
-Wire Wire Line
 	28200 20100 28200 20300
 Connection ~ 28200 20100
@@
 	29150 20150 28500 20150
 Wire Wire Line
-	28500 20150 28500 20050
-Wire Wire Line
 	28500 20150 28500 20300
 Connection ~ 28500 20150
@@
 	29350 20200 28800 20200
 Wire Wire Line
-	28800 20200 28800 20050
-Wire Wire Line
 	28800 20200 28800 20300
 Connection ~ 28800 20200
@@
 	25650 20000 25400 20000
 $Comp
-L Device:R R149
-U 1 1 6C3798DA
-P 25100 19900
-F 0 "R149" H 25170 19946 50  0000 L CNN
-F 1 "4.7k" H 25170 19855 50  0000 L CNN
-F 2 "Resistor_SMD:R_0603_1608Metric" V 25030 19900 50  0001 C CNN
-F 3 "~" H 25100 19900 50  0001 C CNN
-	1    25100 19900
-	1    0    0    -1
-$EndComp
-$Comp
-L Device:R R148
-U 1 1 6C3798E0
-P 24800 19900
-F 0 "R148" H 24870 19946 50  0000 L CNN
-F 1 "4.7k" H 24870 19855 50  0000 L CNN
-F 2 "Resistor_SMD:R_0603_1608Metric" V 24730 19900 50  0001 C CNN
-F 3 "~" H 24800 19900 50  0001 C CNN
-	1    24800 19900
-	1    0    0    -1
-$EndComp
-$Comp
-L Device:R R147
-U 1 1 6C3798E6
-P 24500 19900
-F 0 "R147" H 24570 19946 50  0000 L CNN
-F 1 "4.7k" H 24570 19855 50  0000 L CNN
-F 2 "Resistor_SMD:R_0603_1608Metric" V 24430 19900 50  0001 C CNN
-F 3 "~" H 24500 19900 50  0001 C CNN
-	1    24500 19900
-	1    0    0    -1
-$EndComp
-$Comp
 L Device:R R153
 U 1 1 6C3798EC
 P 24500 20450
 F 0 "R153" H 24570 20496 50  0000 L CNN
-F 1 "4.7k" H 24570 20405 50  0000 L CNN
+F 1 "10k" H 24570 20405 50  0000 L CNN
 F 2 "Resistor_SMD:R_0603_1608Metric" V 24430 20450 50  0001 C CNN
 F 3 "~" H 24500 20450 50  0001 C CNN
@@
 P 24800 20450
 F 0 "R154" H 24870 20496 50  0000 L CNN
-F 1 "4.7k" H 24870 20405 50  0000 L CNN
+F 1 "10k" H 24870 20405 50  0000 L CNN
 F 2 "Resistor_SMD:R_0603_1608Metric" V 24730 20450 50  0001 C CNN
 F 3 "~" H 24800 20450 50  0001 C CNN
@@
 P 25100 20450
 F 0 "R155" H 25170 20496 50  0000 L CNN
-F 1 "4.7k" H 25170 20405 50  0000 L CNN
+F 1 "10k" H 25170 20405 50  0000 L CNN
 F 2 "Resistor_SMD:R_0603_1608Metric" V 25030 20450 50  0001 C CNN
 F 3 "~" H 25100 20450 50  0001 C CNN
@@
 	25400 20100 24500 20100
 Wire Wire Line
-	24500 20100 24500 20050
-Wire Wire Line
 	24500 20100 24500 20300
 Connection ~ 24500 20100
@@
 	25450 20150 24800 20150
 Wire Wire Line
-	24800 20150 24800 20050
-Wire Wire Line
 	24800 20150 24800 20300
 Connection ~ 24800 20150
@@
 	25650 20200 25100 20200
 Wire Wire Line
-	25100 20200 25100 20050
-Wire Wire Line
 	25100 20200 25100 20300
 Connection ~ 25100 20200
@@
 	25800 2650 25800 2600
 Connection ~ 25950 2650
+$Comp
+L Device:Jumper_NO_Small JP2
+U 1 1 62719069
+P 24500 19900
+F 0 "JP2" V 24454 19948 50  0000 L CNN
+F 1 "NO" V 24545 19948 50  0000 L CNN
+F 2 "Jumper:SolderJumper-2_P1.3mm_Open_RoundedPad1.0x1.5mm" H 24500 19900 50  0001 C CNN
+F 3 "~" H 24500 19900 50  0001 C CNN
+	1    24500 19900
+	0    1    1    0
+$EndComp
+Wire Wire Line
+	24500 19800 24500 19750
+Wire Wire Line
+	24500 20000 24500 20100
+Wire Wire Line
+	24800 19800 24800 19750
+Wire Wire Line
+	24800 20000 24800 20150
+Wire Wire Line
+	25100 19800 25100 19750
+Wire Wire Line
+	25100 20000 25100 20200
+Wire Wire Line
+	28800 19800 28800 19750
+Wire Wire Line
+	28800 20000 28800 20200
+Wire Wire Line
+	28500 20000 28500 20150
+Wire Wire Line
+	28500 19800 28500 19750
+Wire Wire Line
+	28200 20000 28200 20100
+Wire Wire Line
+	28200 19800 28200 19750
+$Comp
+L Device:Jumper_NO_Small JP3
+U 1 1 6470FB78
+P 24800 19900
+F 0 "JP3" V 24754 19948 50  0000 L CNN
+F 1 "NO" V 24845 19948 50  0000 L CNN
+F 2 "Jumper:SolderJumper-2_P1.3mm_Open_RoundedPad1.0x1.5mm" H 24800 19900 50  0001 C CNN
+F 3 "~" H 24800 19900 50  0001 C CNN
+	1    24800 19900
+	0    1    1    0
+$EndComp
+$Comp
+L Device:Jumper_NO_Small JP4
+U 1 1 648A76A7
+P 25100 19900
+F 0 "JP4" V 25054 19948 50  0000 L CNN
+F 1 "NO" V 25145 19948 50  0000 L CNN
+F 2 "Jumper:SolderJumper-2_P1.3mm_Open_RoundedPad1.0x1.5mm" H 25100 19900 50  0001 C CNN
+F 3 "~" H 25100 19900 50  0001 C CNN
+	1    25100 19900
+	0    1    1    0
+$EndComp
+$Comp
+L Device:Jumper_NO_Small JP5
+U 1 1 64D6E656
+P 28200 19900
+F 0 "JP5" V 28154 19948 50  0000 L CNN
+F 1 "NO" V 28245 19948 50  0000 L CNN
+F 2 "Jumper:SolderJumper-2_P1.3mm_Open_RoundedPad1.0x1.5mm" H 28200 19900 50  0001 C CNN
+F 3 "~" H 28200 19900 50  0001 C CNN
+	1    28200 19900
+	0    1    1    0
+$EndComp
+$Comp
+L Device:Jumper_NO_Small JP6
+U 1 1 64F06139
+P 28500 19900
+F 0 "JP6" V 28454 19948 50  0000 L CNN
+F 1 "NO" V 28545 19948 50  0000 L CNN
+F 2 "Jumper:SolderJumper-2_P1.3mm_Open_RoundedPad1.0x1.5mm" H 28500 19900 50  0001 C CNN
+F 3 "~" H 28500 19900 50  0001 C CNN
+	1    28500 19900
+	0    1    1    0
+$EndComp
+$Comp
+L Device:Jumper_NO_Small JP7
+U 1 1 6509DC40
+P 28800 19900
+F 0 "JP7" V 28754 19948 50  0000 L CNN
+F 1 "NO" V 28845 19948 50  0000 L CNN
+F 2 "Jumper:SolderJumper-2_P1.3mm_Open_RoundedPad1.0x1.5mm" H 28800 19900 50  0001 C CNN
+F 3 "~" H 28800 19900 50  0001 C CNN
+	1    28800 19900
+	0    1    1    0
+$EndComp
 $EndSCHEMATC
